File: hh2019_proto_rev1_0_0.brd (EAGLE design)
At the start: 95 x 86 mm, 201 parts, among them IC1 CP210X_USB_UART, IC2 LD117AS33TR, IC3 ESP32WROOM32, IC4 TP4056, M1 MOTOR10MM, Q1 MMBT2222A, Q2 MMBT2222A, Q3 MMBT2222A, Q4 MMBT2222A, Q5 SI1304 BDL, Q6 MMBT2222A, U1 MPR121QR2, X2 2908-05WB-MG, X4 JST-PH3

Commit message: Initialised fork from SHA2017 for HackerHotel 2019
Parts:
- added C42, C46: 1u, hh2019_rev0_1_0_dev:C0603-DASHES
- added R26: 0R, hh2019_rev0_1_0_dev:R0603-DASHES
- C1, C10, C11, C12, C14, C16, C19, C2, C21, C22, C23, C25, C27, C28, C29, C3, C31, C32, C33, C35, C36, C37, C38, C39, C4, C40, C44, C45, C5, C6, C7, C8: device sha2017_rev0_1_0_dev:C0603-DASHES -> hh2019_rev0_1_0_dev:C0603-DASHES
- F1, F2: value 900mA -> 1A
- IC2: value LD117AS33TR -> AP2114H
- L1: value 22µ -> 47µ
- R1, R12, R13, R14, R15, R16, R17, R18, R20, R21, R22, R23, R24, R25, R29, R3, R31, R32, R35, R36, R37, R4, R6, R7: device sha2017_rev0_1_0_dev:R0603-DASHES -> hh2019_rev0_1_0_dev:R0603-DASHES
- R19: value 5R -> 2R7; device sha2017_rev0_1_0_dev:R0603-DASHES -> hh2019_rev0_1_0_dev:R0603-DASHES
- R30: value 0R27 -> 0R27 1/4W
- moved $$U$2 1.32 mm to (90.6, 30.0)
- moved U$17 1.17 mm to (88.6, 6.10)
- moved C33 0.90 mm to (76.2, 54.2)
- moved $$U$9 0.81 mm to (50.8, 39.1)
- moved C35 0.70 mm to (76.2, 52.6)
- moved C38 0.50 mm to (76.2, 51.0)
- moved C32 0.10 mm to (72.7, 55.5)
- turned C7 to 180 degrees
Connections:
- new net LCD_VDD: C42.1, R26.2, X1.7
- net +3V3: now also C46.1, R26.1; no longer X1.7
- net GND: now also C42.2, C46.2
Routing:
- net I2C_INT: track 75.4 -> 59.0 mm
- net LCD_VDD: track 0.00 -> 5.71 mm
- net EXTIO-4: track 37.4 -> 33.7 mm, vias 4 -> 2
- net VIBRATOR: track 93.2 -> 90.1 mm
- net GND: track 42.1 -> 44.6 mm, vias 303 -> 308
- net N$44: track 44.3 -> 42.0 mm
- net CHRG_STAT: track 39.9 -> 37.6 mm
- net SD_CD: track 58.6 -> 60.2 mm
- net +3V3: track 233.0 -> 231.4 mm
- net ESP32_FLASH: track 50.7 -> 52.2 mm, vias 4 -> 3
- net PREVGH: track 11.1 -> 12.1 mm
- net 3V3_SWITCHED: track 107.8 -> 107.0 mm
- net VCOM: track 3.71 -> 4.54 mm
- net VSL: track 3.37 -> 4.12 mm
- net WS2812_POWER_EN: track 130.4 -> 129.7 mm
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Other:
- board text added: "Brought to you by: Anne Jan Brouwer Bas van Sisseren Gavan Fantom Jeroen Domburg Markus Bechtold Niek Blankers Sebastian Oort Thomas Roos"
- board text added: "CAUTION: DO NOT LOOK INTO LEDS WITH REMAINING EYE"
- board text added: "Do not touch"
- board text added: "Still Hacking Anyway"
- board text added: "hh2019"
- board text added: "https://hh2019.org/"
- board text removed: "https://sha2017.org/"
