File: hh2019_proto_rev1_0_0.sch (EAGLE design)
At the start: 204 parts, among them IC1 CP210X_USB_UART, IC2 AP2114H, IC3 ESP32WROOM32, IC4 TP4056, M1 MOTOR10MM, Q1 MMBT2222A, Q2 MMBT2222A, Q3 MMBT2222A, Q4 MMBT2222A, Q5 SI1304 BDL, Q6 MMBT2222A, T1 MOSFET-PCHANNEL, T2 MOSFET-PCHANNEL, T3 MOSFET-PCHANNEL, U1 MPR121QR2, X2 2908-05WB-MG, X4 JST-PH3

Commit message: Initialised fork from SHA2017 for HackerHotel 2019
Parts:
- C1, C10, C11, C12, C14, C16, C19, C2, C21, C22, C23, C25, C27, C28, C29, C3, C31, C32, C33, C35, C36, C37, C38, C39, C4, C40, C42, C44, C45, C46, C5, C6, C7, C8: device sha2017_rev0_1_0_dev:C0603-DASHES -> hh2019_rev0_1_0_dev:C0603-DASHES
- R1, R12, R13, R14, R15, R16, R17, R18, R19, R20, R21, R22, R23, R24, R25, R26, R29, R3, R31, R32, R35, R36, R37, R4, R6, R7: device sha2017_rev0_1_0_dev:R0603-DASHES -> hh2019_rev0_1_0_dev:R0603-DASHES
Other:
- note added: "hh2019 Badge"
- note removed: "SHA2017 Badge"
