File: hh2019_proto.sch (EAGLE design)
At the start: 124 parts, among them IC1 CP210X_USB_UART, IC2 AP2114H, IC4 TP4056, J1 PJ-313D, P1 B4B-PH-SM4-TB, Q1 MMBT2222A, Q3 MMBT2222A, Q4 MMBT2222A, Q5 SI1304 BDL, T1 MOSFET-PCHANNEL, T2 MOSFET-PCHANNEL, U1 MPR121QR2, U2 ESP32-WROVER-I, U3 PCM5102A, X4 JST-PH3

Commit message: Finished design, exported BOM and centroid files, and created gerbers
Parts:
- removed Q2: (no value), transistor-power:N-MOSFET-SO8S
- added Q6: SI1304 BDL, SparkFun-DiscreteSemi:MOSFET-NCHANNEL2N7002PW
- renumbered JP2 to BUZZ1, LED1 to IR_LED
Connections:
- net BUZZER: now also Q6.G; no longer Q2.G
- net BUZZ_OUT: now also Q6.D; no longer Q2.D
- net GND: now also Q6.S; no longer Q2.S
Changed lines of the file:
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@@
 </part>
 <part name="IR_R" library="pinhead" library_urn="urn:adsk.eagle:library:325" deviceset="PINHD-1X3" device="" package3d_urn="urn:adsk.eagle:package:22458/2"/>
-<part name="LED1" library="led" library_urn="urn:adsk.eagle:library:259" deviceset="LED" device="5MM" package3d_urn="urn:adsk.eagle:package:15799/2"/>
-<part name="Q2" library="transistor-power" library_urn="urn:adsk.eagle:library:400" deviceset="N-MOSFET-SO8" device="S" package3d_urn="urn:adsk.eagle:package:29505/2"/>
+<part name="IR_LED" library="led" library_urn="urn:adsk.eagle:library:259" deviceset="LED" device="5MM" package3d_urn="urn:adsk.eagle:package:15799/2"/>
 <part name="R5" library="hh2019_proto" deviceset="R0603-DASHES" device="" value="10k">
 <attribute name="MF" value=""/>
@@
 <attribute name="PARTNO" value="ERJ-3GEYJ103V"/>
 </part>
-<part name="JP2" library="pinhead" library_urn="urn:adsk.eagle:library:325" deviceset="PINHD-1X2" device="" package3d_urn="urn:adsk.eagle:package:22435/2"/>
+<part name="BUZZ1" library="pinhead" library_urn="urn:adsk.eagle:library:325" deviceset="PINHD-1X2" device="" package3d_urn="urn:adsk.eagle:package:22435/2"/>
 <part name="SHITTY-ADDON" library="pinhead" library_urn="urn:adsk.eagle:library:325" deviceset="PINHD-2X2" device="" package3d_urn="urn:adsk.eagle:package:22455/2"/>
 <part name="P1" library="B4B-PH-SM4-TB" deviceset="B4B-PH-SM4-TB" device=""/>
+<part name="Q6" library="SparkFun-DiscreteSemi" deviceset="MOSFET-NCHANNEL" device="2N7002PW" value="SI1304 BDL">
+<attribute name="PARTNO" value="SI1308EDL-T1-GE3"/>
+</part>
 </parts>
 <sheets>
@@
 <attribute name="VALUE" x="260.35" y="127" size="1.778" layer="96"/>
 </instance>
-<instance part="LED1" gate="G$1" x="259.08" y="121.92" smashed="yes" rot="R90">
+<instance part="IR_LED" gate="G$1" x="259.08" y="121.92" smashed="yes" rot="R90">
 <attribute name="NAME" x="263.652" y="125.476" size="1.778" layer="95" rot="R180"/>
 <attribute name="VALUE" x="263.652" y="127.635" size="1.778" layer="96" rot="R180"/>
-</instance>
-<instance part="Q2" gate="G$1" x="302.26" y="134.62" smashed="yes">
-<attribute name="NAME" x="307.34" y="137.16" size="1.778" layer="95"/>
-<attribute name="VALUE" x="307.34" y="134.62" size="1.778" layer="96"/>
 </instance>
 <instance part="R5" gate="G$1" x="251.46" y="142.24" smashed="yes">
@@
 <attribute name="PARTNO" x="251.46" y="142.24" size="1.778" layer="96" rot="MR270" display="off"/>
 </instance>
-<instance part="JP2" gate="G$1" x="304.8" y="114.3" smashed="yes">
+<instance part="BUZZ1" gate="G$1" x="304.8" y="114.3" smashed="yes">
 <attribute name="NAME" x="298.45" y="120.015" size="1.778" layer="95"/>
 <attribute name="VALUE" x="298.45" y="109.22" size="1.778" layer="96"/>
@@
 <attribute name="NAME" x="255.26641875" y="78.73856875" size="1.27071875" layer="95" rot="R90"/>
 <attribute name="VALUE" x="269.249040625" y="78.736990625" size="1.271509375" layer="96" rot="R90"/>
+</instance>
+<instance part="Q6" gate="G$1" x="302.26" y="134.62" smashed="yes" rot="MR0">
+<attribute name="PARTNO" x="302.26" y="134.62" size="1.778" layer="96" rot="MR0" display="off"/>
+<attribute name="NAME" x="297.18" y="137.16" size="1.778" layer="95" rot="MR0"/>
+<attribute name="VALUE" x="297.18" y="134.62" size="1.778" layer="96" rot="MR0"/>
 </instance>
 </instances>
@@
 </segment>
 <segment>
-<pinref part="LED1" gate="G$1" pin="C"/>
+<pinref part="IR_LED" gate="G$1" pin="C"/>
 <wire x1="264.16" y1="121.92" x2="266.7" y2="121.92" width="0.1524" layer="91"/>
 <label x="266.7" y="121.92" size="1.778" layer="95"/>
-</segment>
-<segment>
-<pinref part="Q2" gate="G$1" pin="S"/>
-<wire x1="304.8" y1="129.54" x2="304.8" y2="127" width="0.1524" layer="91"/>
-<label x="304.8" y="127" size="1.778" layer="95"/>
 </segment>
 <segment>
@@
 <wire x1="265.43" y1="66.04" x2="256.54" y2="66.04" width="0.1524" layer="91"/>
 <label x="256.54" y="66.04" size="1.778" layer="95" rot="R180"/>
+</segment>
+<segment>
+<pinref part="Q6" gate="G$1" pin="S"/>
+<wire x1="302.26" y1="129.54" x2="302.26" y2="127" width="0.1524" layer="91"/>
+<label x="302.26" y="127" size="1.778" layer="95"/>
 </segment>
 </net>
@@
 </segment>
 <segment>
-<pinref part="JP2" gate="G$1" pin="2"/>
+<pinref part="BUZZ1" gate="G$1" pin="2"/>
 <wire x1="302.26" y1="114.3" x2="292.1" y2="114.3" width="0.1524" layer="91"/>
 <label x="292.1" y="114.3" size="1.778" layer="95" rot="R180"/>
@@
 </segment>
 <segment>
-<pinref part="LED1" gate="G$1" pin="A"/>
+<pinref part="IR_LED" gate="G$1" pin="A"/>
 <wire x1="256.54" y1="121.92" x2="254" y2="121.92" width="0.1524" layer="91"/>
 <label x="254" y="121.92" size="1.778" layer="95" rot="R180"/>
@@
 </segment>
 <segment>
-<pinref part="Q2" gate="G$1" pin="G"/>
-<wire x1="299.72" y1="132.08" x2="297.18" y2="132.08" width="0.1524" layer="91"/>
-<label x="297.18" y="132.08" size="1.778" layer="95" rot="R180"/>
+<pinref part="Q6" gate="G$1" pin="G"/>
+<wire x1="309.88" y1="134.62" x2="312.42" y2="134.62" width="0.1524" layer="91"/>
+<label x="312.42" y="134.62" size="1.778" layer="95"/>
 </segment>
 </net>
 <net name="BUZZ_OUT" class="0">
 <segment>
-<pinref part="Q2" gate="G$1" pin="D"/>
-<wire x1="304.8" y1="139.7" x2="304.8" y2="142.24" width="0.1524" layer="91"/>
-<label x="304.8" y="142.24" size="1.778" layer="95"/>
-</segment>
-<segment>
-<pinref part="JP2" gate="G$1" pin="1"/>
+<pinref part="BUZZ1" gate="G$1" pin="1"/>
 <wire x1="302.26" y1="116.84" x2="292.1" y2="116.84" width="0.1524" layer="91"/>
 <label x="292.1" y="116.84" size="1.778" layer="95" rot="R180"/>
 </segment>
-</net>
+<segment>
+<pinref part="Q6" gate="G$1" pin="D"/>
+<wire x1="302.26" y1="139.7" x2="302.26" y2="142.24" width="0.1524" layer="91"/>
+<label x="302.26" y="142.24" size="1.778" layer="95"/>
+</segment>
+</net>
